Commit message: feat(denis): switch to the ackermann steering controller

File: description/ros2_control/carlikebot.ros2_control.xacro (robot description, xacro)
@@ -8,12 +8,21 @@
         <param name="example_param_hw_stop_duration_sec">3.0</param>
       </hardware>
-      <joint name="${prefix}virtual_front_wheel_joint">
+      <joint name="${prefix}front_right_wheel_joint">
         <command_interface name="position"/>
         <state_interface name="position"/>
       </joint>
-      <joint name="${prefix}virtual_rear_wheel_joint">
+      <joint name="${prefix}front_left_wheel_joint">
+        <command_interface name="position"/>
+        <state_interface name="position"/>
+      </joint>
+      <joint name="${prefix}rear_right_wheel_joint">
         <command_interface name="velocity"/>
+        <state_interface name="position"/>
         <state_interface name="velocity"/>
+      </joint>
+      <joint name="${prefix}rear_left_wheel_joint">
+        <command_interface name="velocity"/>
         <state_interface name="position"/>
+        <state_interface name="velocity"/>
       </joint>
     </ros2_control>
