Commit message: feat: quick testing setup with hw if

File: ros2_control_demo_description/carlikebot/urdf/carlikebot_description.urdf.xacro (robot description, xacro)
@@ -132,21 +132,20 @@
     <!-- front wheels -->
     <!-- virtual front wheel -->
-    <link name="${prefix}virtual_front_wheel">
-      <visual>
-        <origin xyz="0 0 0" rpy="${PI/2} 0 ${PI/2}"/>
-        <geometry>
-          <cylinder length="0.01" radius="${wheel_radius}"/>
+    <link name="${prefix}steering_rack">
+      <visual>
+        <origin xyz="0 0 0" rpy="0 0 0"/>
+        <geometry>
+          <sphere radius="0.1"/>
         </geometry>
         <material name="invisible"/>
       </visual>
     </link>
-    <joint name="${prefix}virtual_front_wheel_joint" type="revolute">
+    <joint name="${prefix}steering_rack_joint" type="prismatic">
       <parent link="${prefix}chassis_link"/>
-      <child link="${prefix}virtual_front_wheel"/>
+      <child link="${prefix}steering_rack"/>
       <origin xyz="${wheelbase/2} 0 -${base_height/2}" rpy="0 0 ${PI/2}"/>
       <axis xyz="0 0 1"/>
       <limit lower="-0.4" upper="0.4" effort="100.0" velocity="0.0"/>
       <dynamics damping="0.2"/>
-       <mimic joint="${prefix}front_right_wheel_joint" multiplier="1.0" offset="0.0"/>
     </joint>
     <!-- front right wheel -->

File: sb_control/description/ros2_control/carlikebot.ros2_control.xacro (robot description, xacro)
@@ -8,18 +8,9 @@
         <param name="example_param_hw_stop_duration_sec">3.0</param>
       </hardware>
-      <joint name="${prefix}front_right_wheel_joint">
+      <joint name="${prefix}steering_rack_joint">
         <command_interface name="position"/>
         <state_interface name="position"/>
       </joint>
-      <joint name="${prefix}front_left_wheel_joint">
-        <command_interface name="position"/>
-        <state_interface name="position"/>
-      </joint>
-      <joint name="${prefix}rear_right_wheel_joint">
-        <command_interface name="velocity"/>
-        <state_interface name="position"/>
-        <state_interface name="velocity"/>
-      </joint>
-      <joint name="${prefix}rear_left_wheel_joint">
+      <joint name="${prefix}virtual_rear_wheel_joint">
         <command_interface name="velocity"/>
         <state_interface name="position"/>
